File: headers-160m.sch (EAGLE design)
At the start: 13 parts

Commit message: Headers: split C5-6 again, make some TX traces shorter
Parts:
- added C5: 1500p, capacitor-wima:C5/2.5
- C6: value 3000p -> 1500p
- renumbered C5-6 to C6
Connections:
- net GND: now also C5.1, RXIN-2.S, RXOUT-2.S, TXIN-1.S, TXOUT-2.S
- net N$5: now also C5.2
Other:
- moved on the sheet: C12, C2, C3, L7, L8, TXIN-1, TXIN-2, TXOUT-1, TXOUT-2
