File: db9-horizontal-autoband.sch (EAGLE design)
At the start: 19 parts, among them U8 PCA9536

Commit message: Fixed hole size on trimmer cap
Fixed hole size on trimmer cap in library PCA9536.lbr and updated the
two autoband boards to use the corrected package. Package can be
replaced on other boards with the one in this library to fix the
problem. Also moved the text on the horizontal board to the bPlace
layer. Couldn't do this on the smaller board as no where to put it!
Parts:
- CT1, CT2: device rcl:C-TRIMMTZ03 -> PCA9536:C-TRIMMTZ03
Changed lines of the file:
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@@
 </classes>
 <parts>
-<part name="CT1" library="rcl" deviceset="C-TRIMM" device="TZ03" value="60p"/>
-<part name="CT2" library="rcl" deviceset="C-TRIMM" device="TZ03" value="60p"/>
+<part name="CT1" library="PCA9536" deviceset="C-TRIMM" device="TZ03" value="60p"/>
+<part name="CT2" library="PCA9536" deviceset="C-TRIMM" device="TZ03" value="60p"/>
 <part name="L8" library="toroids" deviceset="INDUCTOR" device="T30-2-28AWG-15T" value="T30-2 / 15T"/>
 <part name="L7" library="toroids" deviceset="INDUCTOR" device="T30-2-28AWG-15T" value="T30-2 / 12T"/>
