File: db9smt-autoband.brd (EAGLE design)
At the start: 15 x 30.7 mm, 26 parts, among them CON1 PADONPRINT, CON2 PADONPRINT, CON3 PADONPRINT, CON4 PADONPRINT, CON5 PADONPRINT, CON6 PADONPRINT, CON7 PADONPRINT, CON8 PADONPRINT, CON9 PADONPRINT, IC1 PCA9536

Commit message: Fixed hole size on trimmer cap
Fixed hole size on trimmer cap in library PCA9536.lbr and updated the
two autoband boards to use the corrected package. Package can be
replaced on other boards with the one in this library to fix the
problem. Also moved the text on the horizontal board to the bPlace
layer. Couldn't do this on the smaller board as no where to put it!
Parts:
- added C1: 0.1u, eagle-ltspice:C0603
- CT1, CT2: device rcl:CTRIMTZ03 -> PCA9536:CTRIMTZ03
Connections:
- net GND: now also C1.2
- net N$7: now also C1.1
Routing:
- net N$7: track 17.4 -> 19.3 mm, vias 2 -> 3
Changed lines of the file:
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@@
 <?xml version="1.0" encoding="utf-8"?>
 <!DOCTYPE eagle SYSTEM "eagle.dtd">
-<eagle version="8.1.0">
+<eagle version="7.6.0">
 <drawing>
 <settings>
@@
 <grid distance="19.6850394" unitdist="mil" unit="mil" style="lines" multiple="1" display="no" altdistance="0.1" altunitdist="mm" altunit="mm"/>
 <layers>
-<layer number="1" name="Top" color="4" fill="1" visible="no" active="yes"/>
+<layer number="1" name="Top" color="4" fill="1" visible="yes" active="yes"/>
 <layer number="2" name="Route2" color="1" fill="3" visible="no" active="yes"/>
 <layer number="3" name="Route3" color="4" fill="3" visible="no" active="yes"/>
@@
 <layer number="22" name="bPlace" color="7" fill="1" visible="yes" active="yes"/>
 <layer number="23" name="tOrigins" color="15" fill="1" visible="no" active="yes"/>
-<layer number="24" name="bOrigins" color="15" fill="1" visible="no" active="yes"/>
+<layer number="24" name="bOrigins" color="15" fill="1" visible="yes" active="yes"/>
 <layer number="25" name="tNames" color="7" fill="1" visible="no" active="yes"/>
 <layer number="26" name="bNames" color="7" fill="1" visible="yes" active="yes"/>
@@
 </autorouter>
 <elements>
-<element name="CT1" library="rcl" package="CTRIMTZ03" value="60p" x="9.141" y="21.606" smashed="yes" rot="MR90">
+<element name="CT1" library="PCA9536" package="CTRIMTZ03" value="60p" x="9.141" y="21.606" smashed="yes" rot="MR90">
 <attribute name="NAME" x="12.695" y="20.214" size="1.27" layer="26" rot="MR90"/>
 </element>
-<element name="CT2" library="rcl" package="CTRIMTZ03" value="60p" x="9.141" y="8.864" smashed="yes" rot="MR90">
+<element name="CT2" library="PCA9536" package="CTRIMTZ03" value="60p" x="9.141" y="8.864" smashed="yes" rot="MR90">
 <attribute name="NAME" x="12.772" y="7.372" size="1.27" layer="26" rot="MR90"/>
 </element>
@@
 <attribute name="NAME" x="2.681" y="5.252" size="1.27" layer="26" ratio="10" rot="MR270"/>
 <attribute name="VALUE" x="2.162" y="1.8159" size="0.02" layer="28" rot="MR270"/>
+</element>
+<element name="C1" library="eagle-ltspice" package="C0603" value="0.1u" x="12" y="5.5" smashed="yes" rot="MR270">
+<attribute name="SPICEMODEL" value="NONE" x="12" y="5.5" size="1.778" layer="28" rot="MR270" display="off"/>
+<attribute name="SPICEPREFIX" value="C" x="12" y="5.5" size="1.778" layer="28" rot="MR270" display="off"/>
+<attribute name="NAME" x="14.465" y="6.435" size="1.27" layer="26" rot="MR270"/>
+<attribute name="VALUE" x="13.905" y="6.135" size="1.27" layer="28" rot="MR270"/>
 </element>
 </elements>
@@
 <via x="13.648" y="29.435" extent="1-16" drill="0.6" shape="square"/>
 <via x="5.648" y="19.935" extent="1-16" drill="0.6" shape="square"/>
+<contactref element="C1" pad="2"/>
+<via x="9.648" y="4.735" extent="1-16" drill="0.6" shape="square"/>
 </signal>
 <signal name="N$2">
@@
 <contactref element="CON3" pad="P$1"/>
 <contactref element="IC1" pad="8"/>
-<wire x1="11.741" y1="6.06" x2="9.729" y2="6.06" width="0.4064" layer="1"/>
-<wire x1="9.729" y1="6.06" x2="8.033" y2="7.656" width="0.4064" layer="1"/>
-<wire x1="8.033" y1="7.656" x2="5.894" y2="7.656" width="0.4064" layer="1"/>
-<wire x1="5.894" y1="7.656" x2="5.363" y2="8.587" width="0.4064" layer="1"/>
-<wire x1="5.363" y1="8.587" x2="5.363" y2="10.249" width="0.4064" layer="1"/>
+<wire x1="11.741" y1="6.06" x2="11" y2="6.06" width="0.4064" layer="1"/>
+<wire x1="10.24" y1="6.9" x2="10.229" y2="6.96" width="0.4064" layer="1"/>
+<wire x1="10.229" y1="6.96" x2="8.033" y2="7.556" width="0.4064" layer="1"/>
+<wire x1="8.033" y1="7.556" x2="5.894" y2="7.556" width="0.4064" layer="1"/>
+<wire x1="5.894" y1="7.556" x2="5.363" y2="8.087" width="0.4064" layer="1"/>
+<wire x1="5.363" y1="8.087" x2="5.363" y2="10.249" width="0.4064" layer="1"/>
 <wire x1="5.363" y1="10.249" x2="5.54" y2="10.526" width="0.4064" layer="1"/>
 <via x="5.54" y="10.526" extent="1-16" drill="0.6" shape="square"/>
@@
 <via x="5.386" y="15.235" extent="1-16" drill="0.6" shape="square"/>
 <wire x1="5.386" y1="15.235" x2="2.77" y2="15.235" width="0.4064" layer="1"/>
+<contactref element="C1" pad="1"/>
+<wire x1="12" y1="6.35" x2="10.7" y2="6.85" width="0.4064" layer="16"/>
+<wire x1="10.7" y1="6.85" x2="10.24" y2="6.9" width="0.4064" layer="16"/>
+<via x="10.24" y="6.9" extent="1-16" drill="0.6" shape="square"/>
+<wire x1="10.24" y1="6.9" x2="11" y2="6.06" width="0.4064" layer="1"/>
 </signal>
 <signal name="N$8">
@@
 <contactref element="CON5" pad="P$1"/>
 <contactref element="IC1" pad="7"/>
-<wire x1="11.741" y1="4.79" x2="9.891" y2="4.79" width="0.4064" layer="1"/>
-<wire x1="9.891" y1="4.79" x2="7.756" y2="6.925" width="0.4064" layer="1"/>
+<wire x1="11.741" y1="4.79" x2="8.891" y2="6.29" width="0.4064" layer="1"/>
+<wire x1="8.891" y1="6.29" x2="7.756" y2="6.925" width="0.4064" layer="1"/>
 <wire x1="7.756" y1="6.925" x2="5.54" y2="6.925" width="0.4064" layer="1"/>
 <wire x1="5.54" y1="6.925" x2="2.77" y2="9.695" width="0.4064" layer="1"/>
@@
 <contactref element="3" pad="1"/>
 <wire x1="11.741" y1="2.25" x2="11.634" y2="2.25" width="0.4064" layer="1"/>
-<wire x1="11.634" y1="2.25" x2="11.634" y2="1.108" width="0.4064" layer="1"/>
-<via x="11.634" y="1.108" extent="1-16" drill="0.6" shape="square"/>
-<wire x1="11.634" y1="1.108" x2="11.634" y2="3.047" width="0.4064" layer="16"/>
+<wire x1="11.634" y1="2.25" x2="11.634" y2="1.308" width="0.4064" layer="1"/>
+<via x="11.634" y="1.308" extent="1-16" drill="0.6" shape="square"/>
+<wire x1="11.634" y1="1.308" x2="11.634" y2="3.047" width="0.4064" layer="16"/>
 <wire x1="11.634" y1="3.047" x2="9.141" y2="3.047" width="0.4064" layer="16"/>
 <wire x1="9.141" y1="3.047" x2="9.641" y2="2.978" width="0.4064" layer="16"/>
