File: db9-horizontal-autoband-R1.sch (EAGLE design)
At the start: 19 parts, among them U8 PCA9536

Commit message: Fixed errors on horizontal autoband module
Errors fixed:
- Disconnected DB9 pin 7 to allow for future use
- Added 1mm holes to allow toroids to be tied down
- Moved solder jumpers to make room forholes
- Fixed board title text so that it will actually print
- Adjusted restrict on board edge to be narrower
- Minor text placement fixes
Connections:
- net GND: no longer X1.7
Other:
- note added: "Note: X1 pin 7 reserved for use on future boards"
- note removed: "Note: X1 pin 7 and 8 reserved for use on future active 6m module"
Changed lines of the file:
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@@
 <text x="119.126" y="92.202" size="1.016" layer="91">SCL</text>
 <text x="118.618" y="81.788" size="1.016" layer="91">SDA</text>
-<text x="88.9" y="50.8" size="1.778" layer="91">Note: X1 pin 7 and 8 reserved for use on future active 6m module</text>
+<text x="88.9" y="50.8" size="1.778" layer="91">Note: X1 pin 7 reserved for use on future boards</text>
 </plain>
 <instances>
@@
 <net name="GND" class="0">
 <segment>
-<wire x1="99.06" y1="86.36" x2="99.06" y2="83.82" width="0.1524" layer="91"/>
 <wire x1="99.06" y1="83.82" x2="99.06" y2="78.74" width="0.1524" layer="91"/>
 <pinref part="L4" gate="G$1" pin="2"/>
@@
 <pinref part="X1" gate="G$1" pin="8"/>
 <wire x1="99.06" y1="83.82" x2="104.14" y2="83.82" width="0.1524" layer="91"/>
-<pinref part="X1" gate="G$1" pin="7"/>
-<wire x1="99.06" y1="86.36" x2="104.14" y2="86.36" width="0.1524" layer="91"/>
 <pinref part="X1" gate="G$1" pin="G1"/>
 <wire x1="104.14" y1="93.98" x2="99.06" y2="93.98" width="0.1524" layer="91"/>
-<wire x1="99.06" y1="93.98" x2="99.06" y2="86.36" width="0.1524" layer="91"/>
-<junction x="99.06" y="86.36"/>
+<wire x1="99.06" y1="93.98" x2="99.06" y2="83.82" width="0.1524" layer="91"/>
 <pinref part="X1" gate="G$1" pin="G2"/>
 <wire x1="104.14" y1="78.74" x2="99.06" y2="78.74" width="0.1524" layer="91"/>
